File: depot-oben-eda/depot-oben-eda.kicad_sch (KiCad schematic)
At the start: 12 parts, among them J1 SUPPLY, J2 RPi, J3 Schnapper, Q1 BSP76

Commit message: * Change footprint of BSP76 to have D on Pin 4 * Move silkscreen of supply terminal down * increase GND spoke width
Parts:
- Q1: footprint Package_TO_SOT_SMD:SOT-223 -> Package_TO_SOT_SMD:SOT-223-3_TabPin2
Changed lines of the file:
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@@
 	(title_block
 		(title "Schnapper Ansteuerung")
-		(date "2024-12-08")
-		(rev "1.0")
+		(date "2025-01-27")
+		(rev "1.1")
 		(company "jdav Freiburg")
 	)
@@
 	(label "CHECK"
 		(at 170.18 76.2 0)
-		(fields_autoplaced yes)
 		(effects
 			(font
@@
 	(label "BSP_DRAIN"
 		(at 152.4 101.6 0)
-		(fields_autoplaced yes)
 		(effects
 			(font
@@
 	(label "SWITCH"
 		(at 170.18 68.58 0)
-		(fields_autoplaced yes)
 		(effects
 			(font
@@
 	(label "SWITCH"
 		(at 151.13 138.43 0)
-		(fields_autoplaced yes)
 		(effects
 			(font
@@
 	(label "BSP_DRAIN"
 		(at 201.93 123.19 0)
-		(fields_autoplaced yes)
 		(effects
 			(font
@@
 	(label "CHECK"
 		(at 152.4 104.14 0)
-		(fields_autoplaced yes)
 		(effects
 			(font
@@
 			)
 		)
-		(property "Footprint" "Package_TO_SOT_SMD:SOT-223"
+		(property "Footprint" "Package_TO_SOT_SMD:SOT-223-3_TabPin2"
 			(at 191.135 150.495 0)
 			(effects
